Commit message: .

File: robot_description/robots/robot.urdf (robot description, URDF)
Before this commit: robot export_urdf, 6 links, 5 joints
Links:
- link back_wheel: geometry collision mesh filename=package://robot_description/meshes/back_wheel.STL; visual mesh filename=package://robot_description/meshes/back_wheel.STL
- link base_link: geometry collision mesh filename=package://robot_description/meshes/base_link.STL; visual mesh filename=package://robot_description/meshes/base_link.STL
- link kinect_Link: geometry collision mesh filename=package://robot_description/meshes/kinect_Link.STL; visual mesh filename=package://robot_description/meshes/kinect_Link.STL
- link left_wheel: geometry collision mesh filename=package://robot_description/meshes/left_wheel.STL; visual mesh filename=package://robot_description/meshes/left_wheel.STL
- link lidar_link: geometry collision mesh filename=package://robot_description/meshes/lidar_link.STL; visual mesh filename=package://robot_description/meshes/lidar_link.STL
- link right_wheel: geometry collision mesh filename=package://robot_description/meshes/right_wheel.STL; visual mesh filename=package://robot_description/meshes/right_wheel.STL
