Commit message: .

File: src/robot_description/robots/robot.urdf (robot description, URDF)
Before this commit: robot robot_description, 6 links, 5 joints
Joints:
- removed joint rot1
- removed joint rot2
- added joint wheel_left_joint: type continuous, parent base_link, child left_wheel, origin xyz=0 0.149887301627792 -0.0599999999999983 rpy=-1.5707963267949 0.357463595053736 1.22790071016839E-29, axis 0 0 1
- added joint wheel_right_joint: type continuous, parent base_link, child right_wheel, origin xyz=0 -0.150112698372207 -0.06 rpy=1.57079632679477 1.52790873038023 -1.29473733419683E-13, axis 0 0 -1
